File: PCB/KiCAD/PhloraGCCv2_0_2.kicad_sch (KiCad schematic)
At the start: 105 parts, among them J1 Conn_01x06_Female, J11 Conn_01x02, J14 Conn_01x06, J15 Conn_01x06, J2 Conn_01x02, J3 Conn_01x02, J4 Conn_01x01, J5 Rumble, J6 Conn_01x06, J8 USB_B_Micro, Q1 Q_NMOS_GSD, Q2 Q_PMOS_GDS, Q3 Q_NMOS_GSD, SW1 A, SW10 Dup, SW11 Dright, SW12 Ddown, SW2 B, SW3 X, SW4 Y, SW5 Start, SW6 L, SW7 R, SW8 Z, SW9 Dleft, U1 MCP3002, U10 DRV5055A2xDBZxQ1, U11 DRV5055A2xDBZxQ1, U2 Stickbox_Assembly_Main, U3 MCP3002, U4 DRV5055A2xDBZxQ1, U5 Stickbox_Assembly_CStick, U6 AMS1117-3.3, U7 W25Q128JVS, U8 RP2040, U9 DRV5055A2xDBZxQ1, Y1 Crystal_GND24

Commit message: push to commit
committing the push with this commit
Parts:
- added J9: USB-C, CUI_UJ31-CH-G1-SMT-TR, symbol UJ31-CH-G1-SMT-TR:UJ31-CH-G1-SMT-TR
- added R1 (x2): 5.1k, Resistor_SMD:R_0603_1608Metric, symbol Device:R
Connections:
- net GND: now also J9.A1 (GND), J9.A12 (GND), J9.B1 (GND), J9.B12 (GND), J9.SH1 (SHIELD), J9.SH2 (SHIELD), J9.SH3 (SHIELD), J9.SH4 (SHIELD), J9.SH5 (SHIELD), J9.SH6 (SHIELD), R1.1, R1.1
- net GPIO12 renamed LeftZ
- new net: J9.B5 (CC2), R1.2
- new net: J9.A5 (CC1), R1.2
- new net: J9.A4 (VBUS), J9.A9 (VBUS), J9.B4 (VBUS), J9.B9 (VBUS)
- new net 3V3: J9.A2 (SSTXP1), J9.B2 (SSTXP2)
- new net D+: J9.A6 (DP1), J9.B6 (DP2)
- new net D-: J9.A7 (DN1), J9.B7 (DN2)
- new net Data: J9.A11 (SSRXP2)
Other:
- moved on the sheet: H1, H2, H3, H4, H5, H6, H7, H8, H9, J14
